File: FRED_R2D.kicad_sch (KiCad schematic)
At the start: 85 parts, among them J1 DA15_Receptacle_MountingHoles, J2 RJ45_LED_Shielded, J3 Screw_Terminal_01x07, J4 Conn_01x02_Pin, J5 Conn_01x04, J6 Conn_01x05_Pin, J7 Conn_01x04, Q1 MMBT5551, Q2 MMBT5401, Q3 MMBT5401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

Commit message: Version 1.1 for mfg
Parts:
- removed J4: Conn_01x02_Pin, Connector_PinSocket_2.54mm:PinSocket_1x02_P2.54mm_Vertical, symbol Connector:Conn_01x02_Pin
- removed U4: 74AHC1G86, Package_TO_SOT_SMD:SOT-23-5, symbol 74xGxx:74AHC1G86
- added J4: Conn_01x04_Pin, Connector_Molex:Molex_PicoBlade_53047-0410_1x04_P1.25mm_Vertical, symbol Connector:Conn_01x04_Pin
- added U7: 74AHC1G32, Package_TO_SOT_SMD:SOT-23-5, symbol 74xGxx:74AHC1G32
- R13, R14: value 15K -> 10K; LCSC C22809 -> C25804
- R15, R16: value 10K -> 15K; LCSC C25804 -> C22809
Connections:
- net +12V: now also Q1.3 (C), Q4.3 (C); no longer Q2.2 (E), Q3.2 (E)
- net +5V: now also J4.1 (Pin_1), U7.5 (VCC)
- net AGND: now also Q2.3 (C), Q3.3 (C); no longer Q1.2 (E), Q4.2 (E)
- net DOS: now also U7.1
- net EXC: now also R13.1; no longer R15.1
- net EXC_OUT: now also R15.1; no longer R13.1
- net GND: now also J4.3 (Pin_3), U7.3 (GND)
- net LOT: now also U7.2
- net SWIM_PGM_AND_MENU: now also J4.2 (Pin_2)
- net TRACKING_FAULT: now also U7.4
- net VREF: now also U3.3 (+), U3.5 (+); no longer U3.2 (-), U3.6 (-)
- net ~{EXC}: now also R14.1; no longer R16.1
- net ~{EXC}_OUT: now also R16.1; no longer R14.1
- net at R10.1, R9.2: now also Q2.1 (B); no longer Q4.1 (B)
- net at R3.2, R4.1: now also Q3.1 (B); no longer Q1.1 (B)
- net at R14.2, R16.2: now also U3.6 (-); no longer U3.5 (+)
- net at R7.2, R8.1: now also Q4.1 (B); no longer Q2.1 (B)
- net at R6.2: now also Q3.2 (E); no longer Q1.3 (C)
- net at R1.2, R2.1: now also Q1.1 (B); no longer Q3.1 (B)
- net at R12.2: now also Q2.2 (E); no longer Q4.3 (C)
- net at R5.1: now also Q1.2 (E); no longer Q3.3 (C)
- net at R13.2, R15.2: now also U3.2 (-); no longer U3.3 (+)
- net STM_RST: now reaches C21.2, S1.C, S1.D, U5.4 (NRST)
- net STM_RST: now also J4.4 (Pin_4)
- net at R11.1: now also Q4.2 (E); no longer Q2.3 (C)
